File: Tuning Fork Clock.kicad_pcb (KiCad board)
At the start: 2 copper layers, 73.7 x 143.5 mm, 64 parts, among them J3 Conn_Coaxial, J5 Conn_01x02_Male, J6 Conn_01x08_Male, Q1 BC547, Q2 BC547, Q3 BC547, Q4 BC547, Q5 BC547, Q6 BC547, Q7 BC547, SW1 Rotary_Encoder_Switch, U1 NE555P, U10 TuningFork, U2 ATtiny4313-PU, U3 74HC595, U4 SC39-11YWA, U5 SC39-11YWA, U6 SC39-11YWA, U7 SC39-11YWA, U8 SC39-11YWA, U9 L7805

Commit message: Update to KiCAD 6
Connections:
- U1 pad 5: Net-(U1-Pad5) -> unconnected-(U1-Pad5)
- U1 pad 7: Net-(U1-Pad7) -> unconnected-(U1-Pad7)
- U3 pad 9: Net-(U3-Pad9) -> unconnected-(U3-Pad9)
Routing:
- net SCK: track 112.7 -> 108.9 mm
- net +9V: track 52.4 -> 49.7 mm
- net RST: track 61.4 -> 60.5 mm
- net Clock: track 88.1 -> 87.2 mm
- net +5V: track 471.9 -> 471.0 mm
Other:
- board size 73.7 x 143.5 mm -> 73.7 x 143.8 mm
- net class Default removed
- net class Power removed
